File: hardware/main_pcb_hw5/main_pcb_hw5.kicad_sch (KiCad schematic)
At the start: 25 parts, among them J1 MEGA BOTTOM, J10 GBA_Slot, J3 CART SLOT TOP ROW, J4 CART SLOT FRONT ROW, J6 5V USB, J7 Conn_01x07, J8 EXP2, J9 EXP1, M2_1 Screw_Terminal_01x01, M2_2 Screw_Terminal_01x01, M2_3 Screw_Terminal_01x01, M2_4 Screw_Terminal_01x01, M2_5 Screw_Terminal_01x01, M2_6 Screw_Terminal_01x01, M2_7 Screw_Terminal_01x01, M2_8 Screw_Terminal_01x01, M2_9 Screw_Terminal_01x01, SW1 VOLTAGE, SW2 POWER, U2 DS3231MZ

Commit message: -small mod to routing to no split planes -replace gerber zip -replace pcb renders
Parts:
- C5: footprint Capacitor_SMD:C_0402_1005Metric_Pad0.74x0.62mm_HandSolder -> Capacitor_SMD:C_0603_1608Metric_Pad1.08x0.95mm_HandSolder
- J10: footprint (none) -> !sanni:GBA-SLOT-B
- M2_1, M2_2, M2_3, M2_4, M2_5, M2_6, M2_7, M2_8, M2_9: footprint (none) -> MountingHole:MountingHole_2.2mm_M2_ISO7380_Pad
Changed lines of the file:
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@@
       (effects (font (size 1.27 1.27)) (justify left))
     )
-    (property "Footprint" "" (at 254 55.88 0)
+    (property "Footprint" "MountingHole:MountingHole_2.2mm_M2_ISO7380_Pad" (at 254 55.88 0)
       (effects (font (size 1.27 1.27)) hide)
     )
@@
       (effects (font (size 1.27 1.27)) (justify left))
     )
-    (property "Footprint" "" (at 254 45.72 0)
+    (property "Footprint" "MountingHole:MountingHole_2.2mm_M2_ISO7380_Pad" (at 254 45.72 0)
       (effects (font (size 1.27 1.27)) hide)
     )
@@
       (effects (font (size 1.27 1.27)) (justify left))
     )
-    (property "Footprint" "" (at 254 30.48 0)
+    (property "Footprint" "MountingHole:MountingHole_2.2mm_M2_ISO7380_Pad" (at 254 30.48 0)
       (effects (font (size 1.27 1.27)) hide)
     )
@@
       (effects (font (size 1.27 1.27)) (justify left))
     )
-    (property "Footprint" "" (at 254 40.64 0)
+    (property "Footprint" "MountingHole:MountingHole_2.2mm_M2_ISO7380_Pad" (at 254 40.64 0)
       (effects (font (size 1.27 1.27)) hide)
     )
@@
       (effects (font (size 1.27 1.27)) (justify left))
     )
-    (property "Footprint" "" (at 254 60.96 0)
+    (property "Footprint" "MountingHole:MountingHole_2.2mm_M2_ISO7380_Pad" (at 254 60.96 0)
       (effects (font (size 1.27 1.27)) hide)
     )
@@
       (effects (font (size 1.27 1.27)) (justify left))
     )
-    (property "Footprint" "" (at 254 35.56 0)
+    (property "Footprint" "MountingHole:MountingHole_2.2mm_M2_ISO7380_Pad" (at 254 35.56 0)
       (effects (font (size 1.27 1.27)) hide)
     )
@@
       (effects (font (size 1.27 1.27)) (justify left))
     )
-    (property "Footprint" "" (at 254 50.8 0)
+    (property "Footprint" "MountingHole:MountingHole_2.2mm_M2_ISO7380_Pad" (at 254 50.8 0)
       (effects (font (size 1.27 1.27)) hide)
     )
@@
       (effects (font (size 1.27 1.27)))
     )
-    (property "Footprint" "" (at 171.45 20.32 0)
+    (property "Footprint" "!sanni:GBA-SLOT-B" (at 171.45 20.32 0)
       (effects (font (size 1.27 1.27)) hide)
     )
@@
       (effects (font (size 1.27 1.27)) (justify left))
     )
-    (property "Footprint" "" (at 254 25.4 0)
+    (property "Footprint" "MountingHole:MountingHole_2.2mm_M2_ISO7380_Pad" (at 254 25.4 0)
       (effects (font (size 1.27 1.27)) hide)
     )
@@
       (effects (font (size 1.27 1.27)) (justify left))
     )
-    (property "Footprint" "Capacitor_SMD:C_0402_1005Metric_Pad0.74x0.62mm_HandSolder" (at 254 99.06 0)
+    (property "Footprint" "Capacitor_SMD:C_0603_1608Metric_Pad1.08x0.95mm_HandSolder" (at 254 99.06 0)
       (effects (font (size 1.27 1.27)) hide)
     )
@@
       (effects (font (size 1.27 1.27)) (justify left))
     )
-    (property "Footprint" "" (at 254 20.32 0)
-      (effects (font (size 1.27 1.27)) hide)
-    )
+    (property "Footprint" "MountingHole:MountingHole_2.2mm_M2_ISO7380_Pad" (at 254 20.32 0)
+      (effects (font (size 1.27 1.27)) hide)
+    )
